File: olm-flora-sqw-freescale.brd (EAGLE design)
At the start: 37.3 x 50.8 mm, 33 parts, among them IC1 ATMEGA32U4-AU, IC2 DS3231SN, IC3 MCP73831, IC4 MCP1700-33, J1 AYZ0202, X1 USBSMD, X3 8MHz

Commit message: update
Parts:
- moved IC3 0.57 mm to (9.91, 24.6)
Changed lines of the file:
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@@
 <attribute name="VALUE" x="27.305" y="24.638" size="1.27" layer="27"/>
 </element>
-<element name="IC3" library="SparkFunNew" package="SOT23-5" value="MCP73831" x="9.652" y="24.13" smashed="yes" rot="R270">
-<attribute name="NAME" x="11.811" y="25.019" size="0.4064" layer="25" rot="R270"/>
-<attribute name="VALUE" x="9.4615" y="25.0825" size="0.4064" layer="27" rot="R270"/>
+<element name="IC3" library="SparkFunNew" package="SOT23-5" value="MCP73831" x="9.906" y="24.638" smashed="yes" rot="R270">
+<attribute name="NAME" x="12.065" y="25.527" size="0.4064" layer="25" rot="R270"/>
+<attribute name="VALUE" x="9.7155" y="25.5905" size="0.4064" layer="27" rot="R270"/>
 </element>
 <element name="CHG" library="led" package="CHIPLED_0805" value="0805" x="12.954" y="22.098" smashed="yes" rot="R90">
@@
 <wire x1="12.4320375" y1="28.641521875" x2="11.866353125" y2="31.752790625" width="0" layer="19" extent="1-1"/>
 <wire x1="5.969" y1="27.6098" x2="9.144" y2="32.07" width="0" layer="19" extent="1-1"/>
-<wire x1="8.3519" y1="24.13" x2="5.969" y2="27.6098" width="0" layer="19" extent="1-1"/>
+<wire x1="8.6059" y1="24.638" x2="5.969" y2="27.6098" width="0" layer="19" extent="1-1"/>
 <wire x1="16.957521875" y1="24.1160375" x2="12.4320375" y2="28.641521875" width="0" layer="19" extent="1-1"/>
 <wire x1="18.161" y1="19.332" x2="16.957521875" y2="24.1160375" width="0" layer="19" extent="1-1"/>
@@
 <contactref element="X1" pad="VBUS"/>
 <contactref element="D1" pad="C"/>
-<wire x1="10.927" y1="41.898" x2="10.9521" y2="23.18" width="0" layer="19" extent="1-1"/>
+<wire x1="10.927" y1="41.898" x2="11.2061" y2="23.688" width="0" layer="19" extent="1-1"/>
 <wire x1="29.806" y1="40.894" x2="10.927" y2="41.898" width="0" layer="19" extent="1-1"/>
 <wire x1="28.488" y1="12.878" x2="29.806" y2="40.894" width="0" layer="19" extent="1-1"/>
@@
 <wire x1="10.596" y1="15.24" x2="16.891" y2="19.332" width="0" layer="19" extent="1-16"/>
 <wire x1="6.588" y1="11.54" x2="10.596" y2="15.24" width="0" layer="19" extent="1-16"/>
-<wire x1="8.3519" y1="23.18" x2="10.596" y2="15.24" width="0" layer="19" extent="1-16"/>
+<wire x1="8.6059" y1="23.688" x2="10.596" y2="15.24" width="0" layer="19" extent="1-16"/>
 <wire x1="6.858" y1="2.54" x2="6.588" y2="11.54" width="0" layer="19" extent="1-1"/>
 <wire x1="25.4" y1="2.54" x2="26.996" y2="15.24" width="0" layer="19" extent="16-16"/>
@@
 <contactref element="CHG" pad="C"/>
 <contactref element="IC3" pad="1"/>
-<wire x1="11.904" y1="22.098" x2="8.3519" y2="25.08" width="0" layer="19" extent="1-1"/>
+<wire x1="11.904" y1="22.098" x2="8.6059" y2="25.588" width="0" layer="19" extent="1-1"/>
 </signal>
 <signal name="N$10">
 <contactref element="IC3" pad="5"/>
 <contactref element="RC" pad="2"/>
-<wire x1="9.144" y1="33.97" x2="10.9521" y2="25.08" width="0" layer="19" extent="1-1"/>
+<wire x1="9.144" y1="33.97" x2="11.2061" y2="25.588" width="0" layer="19" extent="1-1"/>
 </signal>
 <signal name="N$11">
