File: olm-flora-sqw-noRTC.brd (EAGLE design)
At the start: 37.3 x 50.8 mm, 33 parts, among them IC1 ATMEGA32U4-AU, IC2 DS3231SN, IC3 MCP73831, IC4 MCP1700-33, J1 AYZ0202, X1 USBSMD, X3 8MHz

Commit message: update
Parts:
- removed C4: 0.1, adafruit:C0805K
- removed IC2: DS3231SN, comfile:SO16W
- removed R3, R4, R5, R6: 10k, adafruit:R0805
- removed U$7: BAT, adafruit:CR1220-SMD
- added SV2: (no value), con-lstb:MA04-1
- moved IC3 6.86 mm to (2.79, 23.9)
- moved CHG 5.11 mm to (8.38, 24.4)
- moved C1 2.81 mm to (28.4, 24.1), turned to 90 degrees
- moved CN2 1.37 mm to (6.10, 16.5), turned to 270 degrees
- moved D1 0.72 mm to (31.0, 23.9), turned to 270 degrees
- moved CON4 0.25 mm to (27.7, 3.81)
- moved IC1 0.25 mm to (18.8, 30.2)
- moved X1 0.25 mm to (31.2, 14.5)
- moved X3 0.25 mm to (18.8, 40.6)
Connections:
- removed net 32KHZ: IC2.1, R6.1
- removed net INT/SQW: IC2.3, R3.1
- removed net SCL: IC2.16, R4.1
- removed net SDA: IC2.15, R5.1
- net GND: no longer C4.2, IC2.10, IC2.11, IC2.12, IC2.13, IC2.5, IC2.6, IC2.7, IC2.8, IC2.9, U$7.-
- net RST: no longer IC2.4
- net VBAT: no longer IC2.14, U$7.+$1, U$7.+$2
- net VCC: no longer C4.1, IC2.2, R3.2, R4.2, R5.2, R6.2
